Commit message: setup rgbd_camera

File: src/vehicle_simulator/urdf/rgbd_camera.urdf.xacro (robot description, xacro)
@@ -1,4 +1,4 @@
 <robot xmlns:xacro="http://www.ros.org/wiki/xacro" name="example">
-  <link name="rgbd_camera">
+  <link name="camera">
     <collision>
       <origin xyz="0 0 0" rpy="0 0 0"/>
@@ -19,6 +19,6 @@
     </inertial>
   </link>
-  <gazebo reference="rgbd_camera">
-    <sensor type="depth" name="rgbd_camera">
+  <gazebo reference="camera">
+    <sensor type="depth" name="camera">
       <update_rate>30.0</update_rate>
       <camera name="head">
@@ -34,5 +34,5 @@
         </clip>
       </camera>
-      <plugin name="rgbd_camera_controller" filename="libgazebo_ros_depth_camera.so">
+      <plugin name="rgbd_camera_controller" filename="libgazebo_ros_openni_kinect.so">
         <alwaysOn>true</alwaysOn>
           <baseline>0.2</baseline>

Commit message: add imu.urdf.xacro

File: src/vehicle_simulator/urdf/rgbd_camera.urdf.xacro (robot description, xacro)
@@ -4,5 +4,5 @@
       <origin xyz="0 0 0" rpy="0 0 0"/>
       <geometry>
-        <box size="0.001 0.001 0.001"/>
+        <box size="0.01 0.01 0.01"/>
       </geometry>
     </collision>
@@ -10,5 +10,5 @@
       <origin xyz="0 0 0" rpy="0 0 0"/>
       <geometry>
-        <box size="0.001 0.001 0.001"/>
+        <box size="0.01 0.01 0.01"/>
       </geometry>
     </visual>
@@ -35,5 +35,5 @@
       </camera>
       <plugin name="rgbd_camera_controller" filename="libgazebo_ros_openni_kinect.so">
-        <alwaysOn>true</alwaysOn>
+          <alwaysOn>true</alwaysOn>
           <baseline>0.2</baseline>
           <cameraName>rgbd_camera</cameraName>
